File: Eagle-Files/Ham-Dip.sch (EAGLE design)
At the start: 14 parts, among them IC1 MAX232ECWE

Commit message: Updates
Parts:
- removed IC1: MAX232ECWE, maxim:MAX232ECWE
- removed S2: reset, SparkFun-Electromechanical:TAC_SWITCHSMD
- removed TRRS: AUDIO-JACK3, SparkFun-Connectors:AUDIO-JACK3
- removed U$1, U$6: 10K, Seeed-Resistor-2016:SMD-RES-10K-1%-1/8W(0805)
- removed X1: (no value), con-subd:F09HP
- added AUDIO-JACK, CW-JACK: TRRS, SparkFun-Connectors:AUDIO-JACK3
- added C10, C7, C8, C9: 1uF, SparkFun-Capacitors:1UF-25V-10%(0805)
- added DB-9: (no value), con-subd:F09HP
- added FEL: reset, SparkFun-Electromechanical:TAC_SWITCHSMD
- added MAX-232: MAX232TSSOP, SparkFun-DigitalIC:MAX232TSSOP
- added R4: 330R, Seeed-Resistor-2016:SMD-RES-220R-5%-1/8W(0805)
- added R5: 10K, Seeed-Resistor-2016:SMD-RES-10K-1%-1/8W(0805)
- C1, C2: value 1uf -> 1uF; device Seeed-Capacitor-2016:CERAMIC-1UF-25V-10%-X7R(0603) -> SparkFun-Capacitors:1UF-25V-10%(0805)
- R3: value 330R -> 10K; device Seeed-Resistor-2016:SMD-RES-220R-5%-1/8W(0805) -> Seeed-Resistor-2016:SMD-RES-10K-1%-1/8W(0805)
Connections:
- removed net GPIO: X1.1
- removed net GPIO-#: TRRS.RING2
- removed net XIO-P0: U$2.XIO-P0, U$5.B
- new net 5V: U$2.VCC-5V@2
- new net ADC: U$2.LRADC
- new net AIN: DB-9.9
- new net CW-KEY-3: CW-JACK.RING2, U$2.XIO-P0
- new net GPIO-1: DB-9.8, U$2.XIO-P5
- new net GPIO-2: DB-9.7, U$2.XIO-P7
- new net N$10: C9.1, MAX-232.V+
- new net N$11: C10.2, MAX-232.V-
- new net N$16: C7.2, MAX-232.C1+
- new net N$17: C8.2, MAX-232.C2+
- new net N$18: C7.1, MAX-232.C1-
- new net N$19: C8.1, MAX-232.C2-
- new net XMIT: U$2.XIO-P6, U$5.B
- net AUDIO-IN: now also AUDIO-JACK.TIP; no longer X1.6
- net AUDIO-OUT: now also AUDIO-JACK.RING1; no longer X1.7
- net CW-KEY-1: now also CW-JACK.TIP, U$2.XIO-P4; no longer TRRS.TIP, U$2.XIO-P2
- net CW-KEY-2: now also CW-JACK.RING1, U$2.XIO-P2; no longer TRRS.RING1, U$2.XIO-P4
- net FEL: now also FEL.1, FEL.2; no longer S2.1, S2.2
- net GND: now also AUDIO-JACK.EARTH, C10.1, CW-JACK.EARTH, DB-9.5, FEL.3, FEL.4, MAX-232.GND; no longer IC1G$1.V-, S2.3, S2.4, TRRS.EARTH, U$2.GND@1, X1.5
- net N$1: now also R4.1; no longer R3.1
- net N$3: now also R3.1; no longer U$6.1
- net N$4: now also R3.2; no longer U$6.2
- net PTT: now also AUDIO-JACK.RING2, DB-9.4, R5.2; no longer U$1.2, X1.4
- net RX: now also MAX-232.R1OUT; no longer IC1G$1.R1OUT
- net RXD: now also DB-9.3, MAX-232.R1IN; no longer IC1G$1.R1IN, X1.3
- net TX: now also MAX-232.T1IN; no longer IC1G$1.T1IN
- net TXD: now also DB-9.2, MAX-232.T1OUT; no longer IC1G$1.T1OUT, X1.2
- net VCC: now also C9.2, MAX-232.VCC, R4.2, R5.1, U$2.VCC3V3@1; no longer R3.2, U$1.1, U$2.VCC-5V@2
Other:
- moved on the sheet: D1, R1, R2, R3

Commit message: Updates
Parts:
- C1, C10, C2, C7, C8, C9: device SparkFun-Capacitors:1UF-25V-10%(0805) -> adafruit:C-USC0805
Other:
- moved on the sheet: C1, C10, C2, C7, C8, C9
Changed lines of the file:
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@@
 <part name="R1" library="Seeed-Resistor-2016" deviceset="SMD-RES-2.2K-5%-1/8W(0805)" device="" value="2.2K"/>
 <part name="R2" library="Seeed-Resistor-2016" deviceset="SMD-RES-2.2K-5%-1/8W(0805)" device="" value="2.2K"/>
-<part name="C1" library="SparkFun-Capacitors" deviceset="1UF-25V-10%(0805)" device="" value="1uF"/>
-<part name="C2" library="SparkFun-Capacitors" deviceset="1UF-25V-10%(0805)" device="" value="1uF"/>
+<part name="C1" library="adafruit" deviceset="C-US" device="C0805" value="1uF"/>
+<part name="C2" library="adafruit" deviceset="C-US" device="C0805" value="1uF"/>
 <part name="DB-9" library="con-subd" deviceset="F09HP" device=""/>
 <part name="GND4" library="supply1" deviceset="GND" device=""/>
@@
 <part name="AUDIO-JACK" library="SparkFun-Connectors" deviceset="AUDIO-JACK3" device="" value="TRRS"/>
 <part name="MAX-232" library="SparkFun-DigitalIC" deviceset="MAX232" device="TSSOP"/>
-<part name="C7" library="SparkFun-Capacitors" deviceset="1UF-25V-10%(0805)" device="" value="1uF"/>
-<part name="C8" library="SparkFun-Capacitors" deviceset="1UF-25V-10%(0805)" device="" value="1uF"/>
-<part name="C9" library="SparkFun-Capacitors" deviceset="1UF-25V-10%(0805)" device="" value="1uF"/>
-<part name="C10" library="SparkFun-Capacitors" deviceset="1UF-25V-10%(0805)" device="" value="1uF"/>
+<part name="C7" library="adafruit" deviceset="C-US" device="C0805" value="1uF"/>
+<part name="C8" library="adafruit" deviceset="C-US" device="C0805" value="1uF"/>
+<part name="C9" library="adafruit" deviceset="C-US" device="C0805" value="1uF"/>
+<part name="C10" library="adafruit" deviceset="C-US" device="C0805" value="1uF"/>
 <part name="GND7" library="supply1" deviceset="GND" device=""/>
 <part name="P+1" library="supply1" deviceset="VCC" device=""/>
@@
 <pinref part="C10" gate="G$1" pin="1"/>
 <pinref part="GND7" gate="1" pin="GND"/>
+<wire x1="17.78" y1="101.6" x2="17.78" y2="104.14" width="0.1524" layer="91"/>
 </segment>
 <segment>
@@
 <pinref part="R2" gate="G$1" pin="2"/>
 <pinref part="U$2" gate="G$1" pin="MICIN1"/>
-<wire x1="162.56" y1="170.18" x2="190.5" y2="170.18" width="0.1524" layer="91"/>
-<junction x="162.56" y="170.18"/>
-<wire x1="163.83" y1="170.18" x2="162.56" y2="170.18" width="0.1524" layer="91"/>
+<wire x1="165.1" y1="170.18" x2="190.5" y2="170.18" width="0.1524" layer="91"/>
+<junction x="165.1" y="170.18"/>
+<wire x1="163.83" y1="170.18" x2="165.1" y2="170.18" width="0.1524" layer="91"/>
 </segment>
 </net>
@@
 <pinref part="C1" gate="G$1" pin="2"/>
 <pinref part="R3" gate="G$1" pin="1"/>
-<wire x1="146.05" y1="170.18" x2="144.78" y2="170.18" width="0.1524" layer="91"/>
+<wire x1="146.05" y1="170.18" x2="147.32" y2="170.18" width="0.1524" layer="91"/>
 </segment>
 </net>
@@
 <pinref part="R1" gate="G$1" pin="2"/>
 <pinref part="C2" gate="G$1" pin="1"/>
-<junction x="154.94" y="170.18"/>
-<wire x1="154.94" y1="170.18" x2="153.67" y2="170.18" width="0.1524" layer="91"/>
+<junction x="157.48" y="170.18"/>
+<wire x1="157.48" y1="170.18" x2="153.67" y2="170.18" width="0.1524" layer="91"/>
 <junction x="153.67" y="170.18"/>
 </segment>
@@
 <segment>
 <pinref part="C1" gate="G$1" pin="1"/>
-<wire x1="137.16" y1="170.18" x2="134.62" y2="170.18" width="0.1524" layer="91"/>
+<wire x1="139.7" y1="170.18" x2="134.62" y2="170.18" width="0.1524" layer="91"/>
 <label x="137.16" y="170.18" size="1.778" layer="95" rot="R180"/>
 </segment>
@@
 <wire x1="17.78" y1="129.54" x2="17.78" y2="124.46" width="0.1524" layer="91"/>
 <pinref part="MAX-232" gate="G$1" pin="VCC"/>
-<wire x1="17.78" y1="124.46" x2="17.78" y2="121.92" width="0.1524" layer="91"/>
 <wire x1="-17.78" y1="124.46" x2="17.78" y2="124.46" width="0.1524" layer="91"/>
-<wire x1="17.78" y1="124.46" x2="17.78" y2="121.92" width="0.1524" layer="91"/>
-<junction x="17.78" y="121.92"/>
+<junction x="17.78" y="124.46"/>
 <junction x="17.78" y="124.46"/>
 </segment>
@@
 <segment>
 <pinref part="MAX-232" gate="G$1" pin="V+"/>
-<wire x1="0" y1="114.3" x2="17.78" y2="114.3" width="0.1524" layer="91"/>
+<wire x1="0" y1="114.3" x2="17.78" y2="116.84" width="0.1524" layer="91"/>
 <pinref part="C9" gate="G$1" pin="1"/>
 </segment>
@@
 <segment>
 <pinref part="MAX-232" gate="G$1" pin="V-"/>
-<wire x1="0" y1="109.22" x2="17.78" y2="109.22" width="0.1524" layer="91"/>
+<wire x1="0" y1="109.22" x2="17.78" y2="111.76" width="0.1524" layer="91"/>
 <pinref part="C10" gate="G$1" pin="2"/>
 </segment>
@@
 <pinref part="MAX-232" gate="G$1" pin="C1+"/>
 <pinref part="C7" gate="G$1" pin="2"/>
-<wire x1="-43.18" y1="116.84" x2="-35.56" y2="116.84" width="0.1524" layer="91"/>
+<wire x1="-43.18" y1="119.38" x2="-35.56" y2="116.84" width="0.1524" layer="91"/>
 </segment>
 </net>
@@
 <pinref part="MAX-232" gate="G$1" pin="C2+"/>
 <pinref part="C8" gate="G$1" pin="2"/>
-<wire x1="-43.18" y1="106.68" x2="-35.56" y2="106.68" width="0.1524" layer="91"/>
+<wire x1="-43.18" y1="109.22" x2="-35.56" y2="106.68" width="0.1524" layer="91"/>
 </segment>
 </net>
@@
 <pinref part="C7" gate="G$1" pin="1"/>
 <pinref part="MAX-232" gate="G$1" pin="C1-"/>
-<wire x1="-43.18" y1="109.22" x2="-35.56" y2="109.22" width="0.1524" layer="91"/>
+<wire x1="-43.18" y1="111.76" x2="-35.56" y2="109.22" width="0.1524" layer="91"/>
 <wire x1="-35.56" y1="109.22" x2="-35.56" y2="111.76" width="0.1524" layer="91"/>
 </segment>
@@
 <pinref part="C8" gate="G$1" pin="1"/>
 <pinref part="MAX-232" gate="G$1" pin="C2-"/>
-<wire x1="-43.18" y1="99.06" x2="-35.56" y2="99.06" width="0.1524" layer="91"/>
+<wire x1="-43.18" y1="101.6" x2="-35.56" y2="99.06" width="0.1524" layer="91"/>
 <wire x1="-35.56" y1="99.06" x2="-35.56" y2="101.6" width="0.1524" layer="91"/>
 </segment>
