File: Eagle-Files/Ham-Dip-V2-003.brd (EAGLE design)
At the start: 41.7 x 61.5 mm, 33 parts, among them U1 DS2431P

Commit message: updates
Parts:
- MIC-LVL: value TC33X -> 1K
- renumbered U$3 to MIC-LVL
Connections:
- removed net CW-KEY-3: CW-JACK.RING2, U$2.CSID3
Changed lines of the file:
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@@
 <layer number="119" name="KAP_TEKEN" color="7" fill="1" visible="no" active="yes"/>
 <layer number="120" name="KAP_MAAT1" color="7" fill="1" visible="no" active="yes"/>
-<layer number="121" name="_tsilk" color="7" fill="1" visible="no" active="yes"/>
-<layer number="122" name="_bsilk" color="7" fill="1" visible="no" active="yes"/>
+<layer number="121" name="_tsilk" color="7" fill="1" visible="yes" active="yes"/>
+<layer number="122" name="_bsilk" color="7" fill="1" visible="yes" active="yes"/>
 <layer number="123" name="tTestmark" color="7" fill="1" visible="no" active="yes"/>
 <layer number="124" name="bTestmark" color="7" fill="1" visible="no" active="yes"/>
@@
 <attribute name="MPN" value="1N4007" x="47" y="2.5" size="1.778" layer="27" display="off"/>
 </element>
-<element name="U$3" library="HalfBakedCircuits" package="TC33X" value="TC33X" x="30.5" y="33.5"/>
+<element name="MIC-LVL" library="HalfBakedCircuits" package="TC33X" value="1K" x="30.5" y="33.5"/>
 <element name="U$4" library="HalfBakedCircuits" package="HAM-DIP" value="HAM-DIP" x="17.5" y="30"/>
 </elements>
@@
 <contactref element="U$1" pad="2"/>
 <contactref element="C7" pad="2"/>
-<contactref element="U$3" pad="P$3"/>
+<contactref element="MIC-LVL" pad="P$3"/>
 <wire x1="55" y1="0.611" x2="62.389" y2="5.984" width="0" layer="19" extent="1-1"/>
 <wire x1="39.8829" y1="1.864259375" x2="55" y2="0.611" width="0" layer="19" extent="1-1"/>
@@
 <wire x1="29.6721" y1="21.904859375" x2="27.9957" y2="24.851259375" width="0" layer="19" extent="1-1"/>
 </signal>
-<signal name="CW-KEY-3">
-<contactref element="CW-JACK" pad="RING2"/>
-<contactref element="U$2" pad="CSID3"/>
-<wire x1="39.8829" y1="9.484259375" x2="30.4329" y2="55.814259375" width="0" layer="19" extent="1-1"/>
-</signal>
 <signal name="XMIT">
 <contactref element="R6" pad="1"/>
@@
 </signal>
 <signal name="N$4">
-<contactref element="U$3" pad="P$2"/>
+<contactref element="MIC-LVL" pad="P$2"/>
 </signal>
 <signal name="N$7">
-<contactref element="U$3" pad="P$1"/>
+<contactref element="MIC-LVL" pad="P$1"/>
 <contactref element="R4" pad="1"/>
 <wire x1="11.8921" y1="19.822059375" x2="29.345" y2="36.9" width="0" layer="19" extent="1-1"/>
