File: Eagle-Files/Ham-Dip-V2-004-A.brd (EAGLE design)
At the start: 41.7 x 61.5 mm, 33 parts, among them U1 DS2431P

Commit message: updates
Parts:
- FEL: value reset -> Flash
- moved R2 43.8 mm to (32.7, 32.6)
- moved C1 41.5 mm to (26.8, 27.1)
- moved R1 41.5 mm to (29.7, 27.1), turned to 180 degrees
- moved C7 40.4 mm to (23.7, 27.1), turned to 180 degrees
- moved U$1 39.4 mm to (25.1, 22.2), turned to 270 degrees
- moved D2 30.9 mm to (29.7, 22.2), turned to 270 degrees
- moved D3 21.9 mm to (31.5, 18.0), turned to 180 degrees
- moved R4 21.4 mm to (29.7, 32.5)
- moved AUDIO_OUT 16.9 mm to (28.9, 30.8)
- moved AUDIO_IN 16.3 mm to (12.6, 30.3)
- moved U1 13.7 mm to (9.78, 18.5)
- moved R6 13.1 mm to (26.7, 32.6)
- moved U$4 11.0 mm to (6.50, 30.0)
- moved MIC-LVL 10.5 mm to (20.0, 33.0), turned to 270 degrees
- moved C6 10.4 mm to (17.9, 27.2), turned to 180 degrees
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- renumbered FEL1 to PWR-ON
Connections:
- net LCD-D2 renamed N$7
- net N$3 renamed HPL
- net RX renamed RX1
- net TX renamed TX1
- removed net CW-KEY-3: CW-JACK.RING2, U$2.CSID3
- new net VCC-5V: U$2.VCC5V@1
- new net VCC3V3: U$2.VCC3V3@1
- net COR: now also U$2.CSID2
- net CW-KEY-2: now also U$2.CSID3; no longer U$2.CSID2
- net GND: no longer FEL.3, PWR-ON.3
- net N$4: now also AUDIO_OUT.6
- net VCC: no longer U$2.VCC5V@1
- net VCC/2: no longer U$2.VCC3V3@1
Routing:
- net PTT: track 0.00 -> 103.4 mm, vias 0 -> 1
- net VCC/2: track 0.00 -> 62.4 mm, vias 0 -> 1
- net VCC: track 0.00 -> 57.3 mm, vias 0 -> 1
- net CW-KEY-2: track 0.00 -> 50.4 mm, vias 0 -> 1
- net AUDIO-IN: track 0.00 -> 48.4 mm, vias 0 -> 3
- net TX1: track 0.00 -> 46.8 mm, vias 0 -> 1
- net CW-KEY-1: track 0.00 -> 45.7 mm, vias 0 -> 1
- net XMIT: track 0.00 -> 44.6 mm
- net AUDIO-OUT: track 0.00 -> 44.0 mm, vias 0 -> 1
- net RX1: track 0.00 -> 40.4 mm, vias 0 -> 1
- net ADC: track 0.00 -> 36.1 mm
- net TW1-SDA: track 0.00 -> 34.5 mm
- net HPL: track 0.00 -> 32.3 mm, vias 0 -> 1
- net TW1-SCK: track 0.00 -> 27.0 mm
- net N$4: track 0.00 -> 23.6 mm, vias 0 -> 1
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