File: Eagle-Files/Ham-Dip-V2-004-A.sch (EAGLE design)
At the start: 33 parts, among them U1 DS2431P

Commit message: updates
Parts:
- removed FEL1: reset, SparkFun-Electromechanical:TAC_SWITCHSMD
- added PWR-ON: reset, SparkFun-Electromechanical:TAC_SWITCHSMD
- FEL: value reset -> Flash
Connections:
- net LCD-D2 renamed N$7
- net N$3 renamed HPL
- net RX renamed RX1
- net TX renamed TX1
- net COR: now also U$2.CSID2
- net CW-KEY-2: now also U$2.CSID3; no longer U$2.CSID2
- net GND: now also PWR-ON.4; no longer FEL.3, FEL1.3, FEL1.4
- net N$4: now also AUDIO_OUT.6
- net PWR-UP: now also PWR-ON.1, PWR-ON.2; no longer FEL1.1, FEL1.2
- net VCC: no longer U$2.VCC-5V@2
- net VCC/2: no longer U$2.VCC3V3@1
Other:
- note added: "AUDIO"
- note added: "GPIO CW-Key & Power"
- note added: "MCU / C.H.I.P"
- note added: "Pin-1 (Grounded)"
- note added: "SERIAL COMMUNICATION"
- moved on the sheet: AUDIO-JACK, AUDIO_IN, AUDIO_OUT, C1, C2, C3, C4, C5, C6, C7, CW-JACK, D1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
